File: oracle/mm.kicad_sch (KiCad schematic)
At the start: 18 parts, among them Q3 SS8050, Q4 AO3407A, U5 NE5532

Commit message: add n_core firmware add e_core firmware stub update PCB
Parts:
- added R12: 10k, Resistor_SMD:R_1206_3216Metric, symbol Device:R_US
- added R26: 1k, Resistor_SMD:R_1206_3216Metric, symbol Device:R_US
Connections:
- net ADC_BAT: now also R12.2, R26.1; no longer U5.1, U5.2 (-)
- net GND: now also R26.2
- new net: R12.1, U5.1, U5.2 (-)
Other:
- moved on the sheet: D25, D26, D27, D28, D29, D30, D31, Q3, Q4, R18, R19, R20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
